File: hw/eagle/Gimbal Controller/gimbal_controller.sch (EAGLE design)
At the start: 32 parts, among them X1 PROG, X3 22-23-2031, X4 MOTOR

Commit message: fixed some stuff
Parts:
- X2: value 22-23-2021 -> BATT
- X3: value 22-23-2031 -> UART
- renumbered BATT to X2
Changed lines of the file:
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@@
 <part name="R6" library="rcl" deviceset="R-US_" device="R0805" value="200"/>
 <part name="X4" library="con-molex" deviceset="22-23-2061" device="" value="MOTOR"/>
-<part name="BATT" library="con-molex" deviceset="22-23-2021" device=""/>
+<part name="X2" library="con-molex" deviceset="22-23-2021" device="" value="BATT"/>
 <part name="SUPPLY7" library="supply2" deviceset="GND" device=""/>
 <part name="SUPPLY8" library="supply2" deviceset="GND" device=""/>
@@
 <part name="C9" library="resistor" deviceset="C-US" device="C0805" value="4.7u"/>
 <part name="SUPPLY23" library="supply2" deviceset="GND" device=""/>
-<part name="X3" library="con-molex" deviceset="22-23-2031" device=""/>
+<part name="X3" library="con-molex" deviceset="22-23-2031" device="" value="UART"/>
 <part name="SUPPLY24" library="supply2" deviceset="GND" device=""/>
 <part name="U$8" library="power" deviceset="AP2114H-3.3" device="" technology="AP2114H"/>
@@
 <instance part="X4" gate="-5" x="175.26" y="101.6"/>
 <instance part="X4" gate="-6" x="175.26" y="99.06"/>
-<instance part="BATT" gate="-1" x="-55.88" y="261.62" rot="R90"/>
-<instance part="BATT" gate="-2" x="-53.34" y="261.62" rot="R90"/>
+<instance part="X2" gate="-1" x="-55.88" y="261.62" rot="R90"/>
+<instance part="X2" gate="-2" x="-53.34" y="261.62" rot="R90"/>
 <instance part="SUPPLY7" gate="GND" x="-139.7" y="254" rot="R270"/>
 <instance part="SUPPLY8" gate="GND" x="-134.62" y="220.98"/>
@@
 <net name="VCC" class="0">
 <segment>
-<pinref part="BATT" gate="-1" pin="S"/>
+<pinref part="X2" gate="-1" pin="S"/>
 <wire x1="-55.88" y1="259.08" x2="-55.88" y2="254" width="0.1524" layer="91"/>
 <label x="-55.88" y="254" size="1.778" layer="95" rot="R180"/>
@@
 <net name="GND" class="0">
 <segment>
-<pinref part="BATT" gate="-2" pin="S"/>
+<pinref part="X2" gate="-2" pin="S"/>
 <wire x1="-53.34" y1="259.08" x2="-53.34" y2="254" width="0.1524" layer="91"/>
 <pinref part="SUPPLY21" gate="GND" pin="GND"/>

Commit message: added some pic24 code
Parts:
- R10: value 1.54k -> 470
- R11, R7, R9: value 2k -> 2.2k
Changed lines of the file:
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@@
 <part name="SUPPLY20" library="supply2" deviceset="GND" device=""/>
 <part name="SUPPLY21" library="supply2" deviceset="GND" device=""/>
-<part name="R7" library="resistor" deviceset="R-US_" device="R0805" value="2k"/>
-<part name="R9" library="resistor" deviceset="R-US_" device="R0805" value="2k"/>
-<part name="R10" library="resistor" deviceset="R-US_" device="R0805" value="1.54k"/>
-<part name="R11" library="resistor" deviceset="R-US_" device="R0805" value="2k"/>
+<part name="R7" library="resistor" deviceset="R-US_" device="R0805" value="2.2k"/>
+<part name="R9" library="resistor" deviceset="R-US_" device="R0805" value="2.2k"/>
+<part name="R10" library="resistor" deviceset="R-US_" device="R0805" value="470"/>
+<part name="R11" library="resistor" deviceset="R-US_" device="R0805" value="2.2k"/>
 <part name="SUPPLY22" library="supply2" deviceset="GND" device=""/>
 <part name="C9" library="resistor" deviceset="C-US" device="C0805" value="4.7u"/>
