File: hw/eagle/Gimbal Controller v2/board.brd (EAGLE design)
At the start: 3 parts

Commit message: gitignore test
Connections:
- net GND: now also U$2.P$12, U$2.P$5
Changed lines of the file:
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@@
 <vertex x="7" y="5"/>
 </polygon>
+<contactref element="U$2" pad="P$5"/>
+<contactref element="U$2" pad="P$12"/>
+<wire x1="13" y1="36.94" x2="18" y2="36.94" width="0" layer="19" extent="1-1"/>
+<wire x1="18" y1="19.16" x2="13" y2="19.16" width="0" layer="19" extent="1-1"/>
 </signal>
 <signal name="N$2">
